Commit message: update again

File: robots/scorpio_arm_description.urdf (robot description, URDF)
Before this commit: robot scorpio_arm_description_v3, 7 links, 6 joints
Links:
- link base_link: geometry collision mesh filename=package://scorpio_arm_description/meshes/base_link.STL; visual mesh filename=package://scorpio_arm_description/meshes/base_link.STL
- link link1: mass 0.462790481374202 -> 0.462790481374203; geometry collision mesh filename=package://scorpio_arm_description/meshes/link1.STL; visual mesh filename=package://scorpio_arm_description/meshes/link1.STL
- link link2: geometry collision mesh filename=package://scorpio_arm_description/meshes/link2.STL; visual mesh filename=package://scorpio_arm_description/meshes/link2.STL
- link link3: geometry collision mesh filename=package://scorpio_arm_description/meshes/link3.STL; visual mesh filename=package://scorpio_arm_description/meshes/link3.STL
- link link4: geometry collision mesh filename=package://scorpio_arm_description/meshes/link4.STL; visual mesh filename=package://scorpio_arm_description/meshes/link4.STL
- link link5: mass 0.0811646525056535 -> 0.0811646525056553; geometry collision mesh filename=package://scorpio_arm_description/meshes/link5.STL; visual mesh filename=package://scorpio_arm_description/meshes/link5.STL
- link link6: mass 0.27456433038843 -> 0.274564330363397; geometry collision mesh filename=package://scorpio_arm_description/meshes/link6.STL; visual mesh filename=package://scorpio_arm_description/meshes/link6.STL
