Commit message: updated again and again

File: urdf/scorpio_arm_description.urdf (robot description, URDF)
Before this commit: robot scorpio_arm_description, 7 links, 6 joints
Links:
- link link5: mass 0.0811646525056553 -> 0.0811653306860937
- link link6: mass 0.274564330363397 -> 0.274564356936121
Joints:
- joint joint1: origin xyz=0 0 0.1115 rpy=1.65436122510606E-24 -2.16239755607771E-34 1.77925042286121E-10 -> xyz=0 0 0.1115 rpy=-1.65436122510606E-24 2.16239755607771E-34 1.77925042286121E-10
- joint joint2: origin xyz=0 -0.00775000309120119 0.314499999923826 rpy=1.57079631696602 1.748803E-18 3.14159265358979 -> xyz=0 0.00775000309120119 0.314499999923826 rpy=1.57079631696602 1.748803E-18 0
- joint joint3: origin xyz=0 0.425000094137017 0.0409999999973247 rpy=0 0 0 -> xyz=0 0.425000094137191 0.0409999999690292 rpy=0 0 0
- joint joint5: origin xyz=1.61883599970582E-05 0.0570007543469901 0.197500000000056 rpy=1.5707963267949 0 0 -> xyz=-1.61883600108297E-05 -0.0575007543564076 0.196500000000001 rpy=1.5707963267949 0 3.14159265358979
- joint joint6: axis 0 0 1 -> 0 0 -1; origin xyz=-3.11288537899817E-05 0.0754015995721986 0.0570028742029768 rpy=-1.5707963267949 -1.04851706378525E-28 -2.11069071793014E-14 -> xyz=-0.0753999562300418 0 0.0575000019805907 rpy=3.14159265358979 -1.5707963267949 0
- joint jointt4: origin xyz=-1.49404937263287E-05 0.227498306290618 -0.0332478801440056 rpy=1.5707963267949 0 3.14159265358979 -> xyz=-1.49404937541016E-05 0.228498306290499 -0.03324788012514 rpy=-1.5707963267949 0 0

Commit message: updated again and again and again

File: urdf/scorpio_arm_description.urdf (robot description, URDF)
Before this commit: robot scorpio_arm_description, 7 links, 6 joints
Links:
- link base_link: mass 2.11601477785116 -> 2.50584431442898
- link link2: mass 0.449203640099021 -> 0.449203640099022
- link link5: mass 0.0811653306860937 -> 0.0811653306860956
- link link6: mass 0.274564356936121 -> 0.186980317446745
Joints:
- removed joint jointt4
- added joint joint4: type revolute, parent link3, child link4, origin xyz=-1.49404937541016E-05 0.228498306290499 -0.03324788012514 rpy=-1.5707963267949 0 0, axis 0 0 1
- joint joint1: type revolute -> continuous

Commit message: updated again 3

File: urdf/scorpio_arm_description.urdf (robot description, URDF)
Before this commit: robot scorpio_arm_description, 7 links, 6 joints
Links:
- link base_link: mass 2.50584431442898 -> 2.11601477785117
- link link2: mass 0.449203640099022 -> 0.449203640099021
- link link5: mass 0.0811653306860956 -> 0.0811653306860937
- link link6: mass 0.186980317446745 -> 0.186980317473291

Commit message: update again4

File: urdf/scorpio_arm_description.urdf (robot description, URDF)
Before this commit: robot scorpio_arm_description, 7 links, 6 joints
Links:
- link link2: mass 0.449203640099021 -> 0.449203640099038
- link link3: mass 0.417553118840387 -> 0.417553087898504
- link link4: mass 0.389829536577821 -> 0.389829532509614
- link link5: mass 0.0811653306860937 -> 0.0811653306860973
- link link6: mass 0.186980317473291 -> 0.186980317490548
Joints:
- joint joint1: origin xyz=0 0 0.1115 rpy=-1.65436122510606E-24 2.16239755607771E-34 1.77925042286121E-10 -> xyz=0 0 0.1115 rpy=0 -1.68946233269676E-34 2.86985925493723E-42; type continuous -> revolute
- joint joint2: axis 0 0 -1 -> 0 1 0; origin xyz=0 0.00775000309120119 0.314499999923826 rpy=1.57079631696602 1.748803E-18 0 -> xyz=0 0.00775000309120119 0.314499999923826 rpy=0 -1.68946233269676E-34 2.86985925493723E-42
- joint joint3: axis 0 0 -1 -> 0 1 0; origin xyz=0 0.425000094137191 0.0409999999690292 rpy=0 0 0 -> xyz=0 -0.0409999957917564 0.425000094540175 rpy=0 -1.68946233269676E-34 2.86985925493723E-42
- joint joint4: origin xyz=-1.49404937541016E-05 0.228498306290499 -0.03324788012514 rpy=-1.5707963267949 0 0 -> xyz=0.0293572423190065 0.0332478823524079 0.226604563890855 rpy=0 -1.68946233269676E-34 2.86985925493723E-42
- joint joint5: axis 0 0 1 -> 0 1 0; origin xyz=-1.61883600108297E-05 -0.0575007543564076 0.196500000000001 rpy=1.5707963267949 0 3.14159265358979 -> xyz=0.0252428183612949 -0.0575007524410362 0.194871882536996 rpy=0 -1.68946233269676E-34 2.86985925493723E-42
- joint joint6: axis 0 0 -1 -> -1 0 0; origin xyz=-0.0753999562300418 0 0.0575000019805907 rpy=3.14159265358979 -1.5707963267949 0 -> xyz=0.020768766695969 0.0575000020152065 0.00352185941324046 rpy=0 -1.68946233269676E-34 2.86985925493723E-42

Commit message: update 5

File: urdf/scorpio_arm_description.urdf (robot description, URDF)
Before this commit: robot scorpio_arm_description, 7 links, 6 joints
Links:
- link link2: mass 0.449203640099038 -> 0.449203640099039
Joints:
- joint joint1: type revolute -> continuous
- joint joint2: type revolute -> continuous
- joint joint3: type revolute -> continuous
- joint joint4: type revolute -> continuous
- joint joint5: type revolute -> continuous
- joint joint6: type revolute -> continuous

Commit message: update again6

File: urdf/scorpio_arm_description.urdf (robot description, URDF)
Before this commit: robot scorpio_arm_description, 7 links, 6 joints
Links:
- link link1: mass 0.462790481374203 -> 0.46279
- link link2: mass 0.449203640099039 -> 0.4492
- link link3: mass 0.417553087898504 -> 0.41755
- link link4: mass 0.389829532509614 -> 0.38983
- link link5: mass 0.0811653306860973 -> 0.081165
- link link6: mass 0.186980317490548 -> 0.18698
Joints:
- joint joint1: origin xyz=0 0 0.1115 rpy=0 -1.68946233269676E-34 2.86985925493723E-42 -> xyz=0 0 0.1115 rpy=0 -1.6895E-34 2.8699E-42
- joint joint2: origin xyz=0 0.00775000309120119 0.314499999923826 rpy=0 -1.68946233269676E-34 2.86985925493723E-42 -> xyz=0 0.00775 0.3145 rpy=0 -1.6895E-34 2.8699E-42
- joint joint3: origin xyz=0 -0.0409999957917564 0.425000094540175 rpy=0 -1.68946233269676E-34 2.86985925493723E-42 -> xyz=0 -0.041 0.425 rpy=0 -1.6895E-34 2.8699E-42
- joint joint4: origin xyz=0.0293572423190065 0.0332478823524079 0.226604563890855 rpy=0 -1.68946233269676E-34 2.86985925493723E-42 -> xyz=0.029357 0.033248 0.2266 rpy=0 -1.6895E-34 2.8699E-42
- joint joint5: origin xyz=0.0252428183612949 -0.0575007524410362 0.194871882536996 rpy=0 -1.68946233269676E-34 2.86985925493723E-42 -> xyz=0.025243 -0.057501 0.19487 rpy=0 -1.6895E-34 2.8699E-42
- joint joint6: origin xyz=0.020768766695969 0.0575000020152065 0.00352185941324046 rpy=0 -1.68946233269676E-34 2.86985925493723E-42 -> xyz=0.020769 0.0575 0.0035219 rpy=0 -1.6895E-34 2.8699E-42

Commit message: update 6

File: urdf/scorpio_arm_description.urdf (robot description, URDF)
Before this commit: robot scorpio_arm_description, 7 links, 6 joints
Links:
- link base_link: mass 2.11601477785117 -> 2.11601478181474
- link link1: mass 0.46279 -> 0.462790481374201
- link link2: mass 0.4492 -> 0.449209187922238
- link link3: mass 0.41755 -> 0.417553087871641
- link link4: mass 0.38983 -> 0.389829530881586
- link link5: mass 0.081165 -> 0.0811653306860956
- link link6: mass 0.18698 -> 0.186980321011871
Joints:
- joint joint1: origin xyz=0 0 0.1115 rpy=0 -1.6895E-34 2.8699E-42 -> xyz=0 0 0.109 rpy=0 -1.68946233269676E-34 2.86985925493723E-42
- joint joint2: origin xyz=0 0.00775 0.3145 rpy=0 -1.6895E-34 2.8699E-42 -> xyz=0 0.00875000311574248 0.316999999914016 rpy=1.65436122510606E-24 -3.85185988877447E-34 -1.77925042286121E-10
- joint joint3: origin xyz=0 -0.041 0.425 rpy=0 -1.6895E-34 2.8699E-42 -> xyz=0.0422907473805048 -0.0409999958029054 0.422890734166716 rpy=-1.65436122510606E-24 2.16239755607771E-34 1.77925042286121E-10
- joint joint4: origin xyz=0.029357 0.033248 0.2266 rpy=0 -1.6895E-34 2.8699E-42 -> xyz=-1.49404937540148E-05 0.0322478823721251 0.228498305973538 rpy=0 -1.68946233269676E-34 2.86985925493723E-42
- joint joint5: origin xyz=0.025243 -0.057501 0.19487 rpy=0 -1.6895E-34 2.8699E-42 -> xyz=-1.61883600107299E-05 -0.0575007524250337 0.19650000056517 rpy=0 -1.68946233269676E-34 2.86985925493723E-42
- joint joint6: origin xyz=0.020769 0.0575 0.0035219 rpy=0 -1.6895E-34 2.8699E-42 -> xyz=0.0753999562300418 0.0575000019805965 0 rpy=0 -1.68946233269676E-34 2.86985925493723E-42
